Commit message: edit joint limits

File: myGym/envs/objects/assembly/urdf/btn.urdf (robot description, URDF)
Before this commit: robot btn, 2 links, 1 joints
Links:
- link body: geometry collision mesh filename=./stl/btn_filled_body.stl scale=0.03 0.03 0.03; visual mesh filename=./stl/btn_filled_body.stl scale=0.03 0.03 0.03
- link stick: mass 10000.0 -> 0.1
Joints:
- joint joint: limit lower=-6.28318530718 upper=6.28318530718 effort=330.0 velocity=2.16 -> lower=-0.03 upper=0 effort=0 velocity=2.16

Commit message: changing btn scale

File: myGym/envs/objects/assembly/urdf/btn.urdf (robot description, URDF)
Before this commit: robot btn, 2 links, 1 joints
Links:
- link body: geometry collision mesh filename=./stl/btn_filled_body.stl scale=0.02 0.02 0.02; visual mesh filename=./stl/btn_filled_body.stl scale=0.02 0.02 0.02
- link stick: mass 0.1 -> 1; geometry collision mesh filename=./stl/btn_press.stl scale=0.02 0.02 0.02; visual mesh filename=./stl/btn_press.stl scale=0.02 0.02 0.02
